File: kicad/terminal/terminal.sch (KiCad schematic (older format))
At the start: 29 parts, among them J1 USB, J2 PS2, J3 VGA, J5 Serial, J6 External 5V, J7 ICSP, U1 PIC32MX270F256B-I_SP, U2 MCP1700-3302E_TO92, Y1 20MHz

Commit message: ground planes instead of traces, fatter traces for power
Parts:
- U1: symbol terminal:PIC32MX270F256B-I_SP -> terminal-rescue:PIC32MX270F256B-I_SP-terminal
Changed lines of the file:
@@
 EESchema Schematic File Version 4
-LIBS:terminal-cache
 EELAYER 30 0
 EELAYER END
@@
 $EndComp
 $Comp
-L terminal:PIC32MX270F256B-I_SP U1
+L terminal-rescue:PIC32MX270F256B-I_SP-terminal U1
 U 1 1 5D617B4B
 P 6250 2400
